Commit message: Updated op point

File: resources/kuka_iiwa/kuka_iiwa.urdf (robot description, URDF)
Before this commit: robot kuka_iiwa, 8 links, 7 joints
Links:
- link link6: mass 1 -> 3.3; geometry visual mesh filename=meshes/daihen_welding_tool.obj scale=1.05 1.05 1.05; visual mesh filename=meshes/link6.obj scale=1 1 1

Commit message: Added stable haptic position feedback

File: resources/kuka_iiwa/kuka_iiwa.urdf (robot description, URDF)
Before this commit: robot kuka_iiwa, 8 links, 7 joints
Links:
- link link6: geometry collision sphere radius=0.005; visual mesh filename=meshes/daihen_welding_tool.obj scale=1.05 1.05 1.05

Commit message: Updated urdf for robot operation

File: resources/kuka_iiwa/kuka_iiwa.urdf (robot description, URDF)
Before this commit: robot kuka_iiwa, 8 links, 7 joints
Links:
- link link6: mass 3.3 -> 2.75

Commit message: Mass commit changes for KUKA real experiment

File: resources/kuka_iiwa/kuka_iiwa.urdf (robot description, URDF)
Before this commit: robot kuka_iiwa, 8 links, 7 joints
Links:
- link link6: mass 2.75 -> 2.445
Joints:
- joint j0: origin xyz=0.000000 0.000000 0.155767 rpy=-0.000000 0.000000 -0.000000 -> xyz=0.000000 0.000000 0.155767 rpy=0.000000 0.000000 0.000000
- joint j1: origin xyz=0.000000 0.000000 0.182500 rpy=-0.000000 0.000000 -0.000000 -> xyz=0.000000 0.000000 0.182500 rpy=0.000000 0.000000 0.000000
- joint j2: origin xyz=0.000000 0.000000 0.185000 rpy=-0.000000 0.000000 -0.000000 -> xyz=0.000000 0.000000 0.185000 rpy=0.000000 0.000000 0.000000
- joint j3: origin xyz=0.000000 0.000000 0.217000 rpy=-0.000000 0.000000 -0.000000 -> xyz=0.000000 0.000000 0.217000 rpy=0.000000 0.000000 3.1415926535897
- joint j4: origin xyz=0.000000 0.000000 0.186000 rpy=-0.000000 0.000000 -0.000000 -> xyz=0.000000 0.000000 0.186000 rpy=0.000000 0.000000 -3.1415926535897
- joint j5: origin xyz=0.000000 0.000000 0.217003 rpy=-0.000000 0.000000 -0.000000 -> xyz=0.000000 0.000000 0.217003 rpy=0.000000 0.000000 0.000000
- joint j6: origin xyz=0.000000 0.000000 0.081000 rpy=-0.000000 0.000000 -0.000000 -> xyz=0.000000 0.000000 0.081000 rpy=0.000000 0.000000 0.000000

Commit message: Switched to TIG torch with demo1

File: resources/kuka_iiwa/kuka_iiwa.urdf (robot description, URDF)
Before this commit: robot kuka_iiwa, 8 links, 7 joints
Links:
- link link6: geometry collision sphere radius=0.003; visual mesh filename=meshes/link6.obj scale=1 1 1
